File: Hardware/Arduino_PCB/Display_Backplate/Display_Backplate_v1/Display_Backplate_v1.kicad_pcb (KiCad board)
At the start: 2 copper layers, 30 x 40 mm, 8 parts, among them J1 Conn_01x14, J2 Conn_02x04_Counter_Clockwise

Commit message: update Display-PCB
Connections:
- J1 pad 1: GND -> +3V3
- J1 pad 2: Net-(J1-Pad2) -> GND
- J2 pad 1: GND -> +3V3
- J2 pad 2: Net-(J1-Pad2) -> GND
Routing:
- net +3V3: track 0.00 -> 38.2 mm
- net Net-(J1-Pad2): track 31.0 -> 0.00 mm
- net GND: track 38.2 -> 31.0 mm
- added copper zone on F.Cu, net +3V3
- removed copper zone on F.Cu, net GND
