File: Hardware/Arduino_PCB/DUE_Shield/DUE_Shield_v1/DUE_Shield_v1.sch (KiCad schematic (older format))
At the start: 33 parts, among them J1 SPI_Header, J3 Reset_+_Dos, J4 V_Supply, J5 Main_Con, J6 Motor_PWM, J7 Audio, J8 Display_Con, J9 Erweiterungs_Con, P1 Digital, P2 Power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

Commit message: Update DUE_Shield inkl. 3d-Modelle
Connections:
- net +5V: now also J6.1 (Pin_1); no longer J6.5 (Pin_5)
- net 10(**): now also J6.4 (Pin_4); no longer J6.2 (Pin_2)
- net 12(**): now also J6.2 (Pin_2); no longer J6.4 (Pin_4)
- net 9(**): now also J6.5 (Pin_5); no longer J6.1 (Pin_1)
Other:
- moved on the sheet: TP7
Changed lines of the file:
@@
 $EndComp
 Wire Wire Line
-	2000 1700 2400 1700
+	2000 2100 2400 2100
+Wire Wire Line
+	2000 2000 2400 2000
+Wire Wire Line
+	2000 1900 2400 1900
 Wire Wire Line
 	2000 1800 2400 1800
-Wire Wire Line
-	2000 1900 2400 1900
-Wire Wire Line
-	2000 2000 2400 2000
-Text Label 2400 1700 2    50   ~ 0
+Text Label 2400 2100 2    50   ~ 0
 9(**)
-Text Label 2400 1800 2    50   ~ 0
+Text Label 2400 2000 2    50   ~ 0
 10(**)
 Text Label 2400 1900 2    50   ~ 0
 11(**)
-Text Label 2400 2000 2    50   ~ 0
+Text Label 2400 1800 2    50   ~ 0
 12(**)
 $Comp
 L power:+5V #PWR0105
 U 1 1 614E0796
-P 2650 2000
-F 0 "#PWR0105" H 2650 1850 50  0001 C CNN
-F 1 "+5V" H 2665 2173 50  0000 C CNN
-F 2 "" H 2650 2000 50  0001 C CNN
-F 3 "" H 2650 2000 50  0001 C CNN
-	1    2650 2000
-	1    0    0    -1
-$EndComp
-Wire Wire Line
-	2650 2000 2650 2100
-Wire Wire Line
-	2650 2100 2000 2100
+P 2650 1600
+F 0 "#PWR0105" H 2650 1450 50  0001 C CNN
+F 1 "+5V" H 2665 1773 50  0000 C CNN
+F 2 "" H 2650 1600 50  0001 C CNN
+F 3 "" H 2650 1600 50  0001 C CNN
+	1    2650 1600
+	1    0    0    -1
+$EndComp
+Wire Wire Line
+	2650 1600 2650 1700
+Wire Wire Line
+	2650 1700 2000 1700
 $Comp
 L Connector_Generic:Conn_01x04 J7
@@
 L Connector:TestPoint TP7
 U 1 1 615B7D82
-P 2800 2000
-F 0 "TP7" H 2858 2118 50  0000 L CNN
-F 1 "TestPoint" H 2858 2027 50  0000 L CNN
-F 2 "TestPoint:TestPoint_Pad_D2.0mm" H 3000 2000 50  0001 C CNN
-F 3 "~" H 3000 2000 50  0001 C CNN
-	1    2800 2000
-	1    0    0    -1
-$EndComp
-Wire Wire Line
-	2800 2000 2800 2100
-Wire Wire Line
-	2800 2100 2650 2100
-Connection ~ 2650 2100
+P 2800 1600
+F 0 "TP7" H 2858 1718 50  0000 L CNN
+F 1 "TestPoint" H 2858 1627 50  0000 L CNN
+F 2 "TestPoint:TestPoint_Pad_D2.0mm" H 3000 1600 50  0001 C CNN
+F 3 "~" H 3000 1600 50  0001 C CNN
+	1    2800 1600
+	1    0    0    -1
+$EndComp
+Wire Wire Line
+	2800 1600 2800 1700
+Wire Wire Line
+	2800 1700 2650 1700
+Connection ~ 2650 1700
 Wire Wire Line
 	2850 5000 3100 5000
